Commit message: added urdfs for matlab

File: include/tiago.urdf (robot description, URDF)
Before this commit: robot tiago, 88 links, 87 joints
Links:
- removed link hand_grasping_frame
- removed link hand_index_abd_link
- removed link hand_index_flex_1_link
- removed link hand_index_flex_2_link
- removed link hand_index_flex_3_link
- removed link hand_index_link
- removed link hand_index_virtual_1_link
- removed link hand_index_virtual_2_link
- removed link hand_index_virtual_3_link
- removed link hand_little_abd_link
- removed link hand_little_flex_1_link
- removed link hand_little_flex_2_link
- removed link hand_little_flex_3_link
- removed link hand_little_virtual_1_link
- removed link hand_little_virtual_2_link
- removed link hand_little_virtual_3_link
- removed link hand_middle_abd_link
- removed link hand_middle_flex_1_link
- removed link hand_middle_flex_2_link
- removed link hand_middle_flex_3_link
- removed link hand_middle_virtual_1_link
- removed link hand_middle_virtual_2_link
- removed link hand_middle_virtual_3_link
- removed link hand_mrl_link
- removed link hand_palm_link
- removed link hand_ring_abd_link
- removed link hand_ring_flex_1_link
- removed link hand_ring_flex_2_link
- removed link hand_ring_flex_3_link
- removed link hand_ring_virtual_1_link
- removed link hand_ring_virtual_2_link
- removed link hand_ring_virtual_3_link
- removed link hand_safety_box
- removed link hand_thumb_abd_link
- removed link hand_thumb_flex_1_link
- removed link hand_thumb_flex_2_link
- removed link hand_thumb_link
- removed link hand_thumb_virtual_1_link
- removed link hand_thumb_virtual_2_link
- link arm_1_link: mass 1.563428 -> None
- link arm_2_link: mass 1.800397 -> None
- link arm_3_link: mass 1.8 -> None
- link arm_4_link: mass 1.432697 -> None
- link arm_5_link: mass 1.655819 -> None
- link arm_6_link: mass 0.370063 -> None
- link arm_7_link: mass 0.234252 -> None
- link arm_tool_link: mass 0.1 -> None
- link base_antenna_left_link: mass 0.000001 -> None
- link base_antenna_right_link: mass 0.000001 -> None
- link base_cover_link: mass 0.25821000000 -> None
- link base_imu_link: mass 0.01 -> None
- link base_laser_link: mass 0.28922000000 -> None
- link base_link: mass 28.26649 -> None
- link base_sonar_01_link: mass 0.001 -> None
- link base_sonar_02_link: mass 0.001 -> None
- link base_sonar_03_link: mass 0.001 -> None
- link caster_back_left_1_link: mass 0.05144761 -> None
- link caster_back_left_2_link: mass 0.08855784 -> None
- link caster_back_right_1_link: mass 0.05144761 -> None
- link caster_back_right_2_link: mass 0.08855784 -> None
- link caster_front_left_1_link: mass 0.05144761 -> None
- link caster_front_left_2_link: mass 0.08855784 -> None
- link caster_front_right_1_link: mass 0.05144761 -> None
- link caster_front_right_2_link: mass 0.08855784 -> None
- link hand_tool_link: mass 0.0001 -> None
- link head_1_link: mass 0.62220 -> None
- link head_2_link: mass 0.66123 -> None
- link head_front_camera_depth_frame: mass 0.001 -> None
- link head_front_camera_depth_optical_frame: mass 0.001 -> None
- link head_front_camera_link: mass 0.21970000000 -> None
- link head_front_camera_optical_frame: mass 0.001 -> None
- link head_front_camera_orbbec_aux_joint_frame: mass 0.001 -> None
- link head_front_camera_rgb_frame: mass 0.001 -> None
- link head_front_camera_rgb_optical_frame: mass 0.001 -> None
- link suspension_left_link: mass 10 -> None
- link suspension_right_link: mass 10 -> None
- link torso_fixed_column_link: mass 0.01 -> None
- link torso_fixed_link: mass 14.01360 -> None
- link torso_lift_link: mass 6.93198 -> None
- link wheel_left_link: mass 1.82362 -> None
- link wheel_right_link: mass 1.82362 -> None
- link wrist_ft_link: mass 0.1 -> None
- link wrist_ft_tool_link: mass 0.1 -> None
Joints:
- removed joint hand_grasping_fixed_joint
- removed joint hand_index_abd_joint
- removed joint hand_index_flex_1_joint
- removed joint hand_index_flex_2_joint
- removed joint hand_index_flex_3_joint
- removed joint hand_index_joint
- removed joint hand_index_virtual_1_joint
- removed joint hand_index_virtual_2_joint
- removed joint hand_index_virtual_3_joint
- removed joint hand_little_abd_joint
- removed joint hand_little_flex_1_joint
- removed joint hand_little_flex_2_joint
- removed joint hand_little_flex_3_joint
- removed joint hand_little_virtual_1_joint
- removed joint hand_little_virtual_2_joint
- removed joint hand_little_virtual_3_joint
- removed joint hand_middle_abd_joint
- removed joint hand_middle_flex_1_joint
- removed joint hand_middle_flex_2_joint
- removed joint hand_middle_flex_3_joint
- removed joint hand_middle_virtual_1_joint
- removed joint hand_middle_virtual_2_joint
- removed joint hand_middle_virtual_3_joint
- removed joint hand_mrl_joint
- removed joint hand_palm_joint
- removed joint hand_ring_abd_joint
- removed joint hand_ring_flex_1_joint
- removed joint hand_ring_flex_2_joint
- removed joint hand_ring_flex_3_joint
- removed joint hand_ring_virtual_1_joint
- removed joint hand_ring_virtual_2_joint
- removed joint hand_ring_virtual_3_joint
- removed joint hand_safety_box_joint
- removed joint hand_thumb_abd_joint
- removed joint hand_thumb_flex_1_joint
- removed joint hand_thumb_flex_2_joint
- removed joint hand_thumb_joint
- removed joint hand_thumb_virtual_1_joint
- removed joint hand_thumb_virtual_2_joint
- joint torso_lift_joint: type prismatic -> fixed
